Commit message: more accurate pi for opw kinematic

File: urdf/SR80.urdf (robot description, URDF)
Before this commit: robot SR80, 11 links, 10 joints
Joints:
- joint J2: origin xyz=0.175 0 0 rpy=1.5708 -1.5708 0 -> xyz=0.175 0 0 rpy=1.570796327 -1.5707963270
- joint J4: origin xyz=0.206 0 0 rpy=1.5708 0 0 -> xyz=0.206 0 0 rpy=1.570796327 0 0
- joint J5: origin xyz=0 0 1.02 rpy=-1.5708 0 0 -> xyz=0 0 1.02 rpy=-1.570796327 0 0
- joint J6: origin xyz=0 -0.25 0 rpy=1.5708 0 0 -> xyz=0 -0.25 0 rpy=1.570796327 0 0

Commit message: typo

File: urdf/SR80.urdf (robot description, URDF)
Before this commit: robot SR80, 11 links, 10 joints
Joints:
- joint J2: origin xyz=0.175 0 0 rpy=1.570796327 -1.5707963270 -> xyz=0.175 0 0 rpy=1.570796327 -1.570796327 0
